File: board/sensor-board/sensor-board.kicad_pcb (KiCad board)
At the start: 2 copper layers, 40 x 40 mm, 16 parts, among them J1 505110-2091

Commit message: minor changes
Parts:
- moved H4 1.43 mm to (135.0, 85.0)
- moved H3 1.42 mm to (135.0, 115.0)
- moved H1 1.41 mm to (165.0, 85.0)
- moved H2 1.40 mm to (165.0, 115.0)
- moved C5 0.31 mm to (147.5, 109.5)
- moved C3 0.19 mm to (145.4, 109.5)
Routing:
- net GNDREF: track 21.5 -> 30.0 mm, vias 8 -> 22
Other:
- board text added: "Sensor Board 0.1.4 2023"
- board text removed: "Sensor Board 0.1.3 2023"
