File: board/board.kicad_pcb (KiCad board)
At the start: 2 copper layers, 60 x 30 mm, 73 parts, among them IC1 NC7SZ11P6X, IC2 FM25L16B-DG, IC3 NCP189CMTW330TAG, J1 USB, J2 Conn_01x12, J3 Conn_01x03, J4 MEM2085-00-115-00-A, SW1 SW_Push, SW2 SW_Push, U1 MT9M001C12STM, U2 APS6404L-3SQR-ZR, U3 RP2350_60QFN, Y1 ABM8-272-T3

Commit message: use embassy
Other:
- board text added: "2025/12"
- board text removed: "2025/10"
Changed lines of the file:
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@@
 		)
 	)
-	(gr_text "2025/10"
+	(gr_text "2025/12"
 		(at 150.65 98.85 0)
 		(layer "B.SilkS")
@@
 			(justify left bottom mirror)
 		)
-		(render_cache "2025/10" 0
+		(render_cache "2025/12" 0
 			(polygon
 				(pts
@@
 			(polygon
 				(pts
-					(xy 139.999423 96.657929) (xy 140.160233 96.708497) (xy 140.30191 96.790745) (xy 140.418215 96.898689)
-					(xy 140.509716 97.029816) (xy 140.577449 97.185564) (xy 140.617806 97.355429) (xy 140.631744 97.544357)
-					(xy 140.61781 97.733305) (xy 140.577449 97.903308) (xy 140.509688 98.058785) (xy 140.418215 98.189231)
-					(xy 140.302017 98.29662) (xy 140.160233 98.379423) (xy 139.999378 98.430586) (xy 139.807791 98.448642)
-					(xy 139.613174 98.430529) (xy 139.451221 98.379423) (xy 139.308966 98.296475) (xy 139.194033 98.189231)
-					(xy 139.10424 98.058841) (xy 139.038292 97.903308) (xy 138.99924 97.733377) (xy 138.985743 97.544357)
-					(xy 139.422644 97.544357) (xy 139.435503 97.722212) (xy 139.470045 97.85725) (xy 139.522027 97.958715)
-					(xy 139.597786 98.038854) (xy 139.691118 98.086487) (xy 139.807791 98.103184) (xy 139.925731 98.086427)
-					(xy 140.019646 98.038737) (xy 140.09546 97.958715) (xy 140.147442 97.85725) (xy 140.181984 97.722212)
-					(xy 140.194842 97.544357) (xy 140.181981 97.3665) (xy 140.147436 97.231523) (xy 140.09546 97.130158)
-					(xy 140.019634 97.050038) (xy 139.925719 97.002301) (xy 139.807791 96.985529) (xy 139.69113 97.002241)
-					(xy 139.597798 97.049921) (xy 139.522027 97.130158) (xy 139.470051 97.231523) (xy 139.435506 97.3665)
-					(xy 139.422644 97.544357) (xy 138.985743 97.544357) (xy 138.999243 97.355357) (xy 139.038292 97.185564)
-					(xy 139.104211 97.029761) (xy 139.194033 96.898689) (xy 139.309074 96.790888) (xy 139.451221 96.708497)
-					(xy 139.613128 96.657986) (xy 139.807791 96.640072)
+					(xy 139.219434 97.210648) (xy 139.232762 97.33532) (xy 139.272142 97.449737) (xy 139.333527 97.556529)
+					(xy 139.416612 97.661838) (xy 139.514873 97.760405) (xy 139.634745 97.860761) (xy 139.908602 98.059526)
+					(xy 139.908602 98.06667) (xy 139.543935 98.052382) (xy 139.077346 98.052382) (xy 139.077346 98.408)
+					(xy 140.583482 98.408) (xy 140.583482 98.151923) (xy 140.22834 97.900133) (xy 139.932575 97.663425)
+					(xy 139.815131 97.548109) (xy 139.730952 97.443704) (xy 139.673893 97.334641) (xy 139.656336 97.233668)
+					(xy 139.662506 97.174526) (xy 139.679515 97.12857) (xy 139.7071 97.089802) (xy 139.744288 97.058399)
+					(xy 139.842083 97.018392) (xy 139.963691 97.00585) (xy 140.094142 97.014948) (xy 140.246121 97.044428)
+					(xy 140.400574 97.091144) (xy 140.565701 97.158258) (xy 140.565701 96.80518) (xy 140.436948 96.74644)
+					(xy 140.281524 96.693732) (xy 140.10308 96.654995) (xy 139.906856 96.640072) (xy 139.759684 96.649759)
+					(xy 139.629506 96.677539) (xy 139.510155 96.724564) (xy 139.412008 96.787241) (xy 139.331187 96.867796)
+					(xy 139.270237 96.965526) (xy 139.232673 97.077265)
 				)
 			)
